File: KiCad/RemoteDevice/RemoteDevice.kicad_pcb (KiCad board)
At the start: 2 copper layers, 93 x 52 mm, 42 parts, among them J1 Alim, J2 CN1, Q1 Si4435, SW1 BP, SW2 BP, U1 XC9140, U2 STM32L041F6Px, U3 MCP6281, U4 ADT7410TRZ, U5 MCP6281, U6 RT606, U7 Microphone

Commit message: Version PCB réalisée au GEI. Des améliorations sont à apporter, voir Amelioration_PCB.txt
Routing:
- net (no net): vias 4 -> 8
Other:
- board size 93 x 52 mm -> 99.5 x 59.2 mm
Changed lines of the file:
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@@
     (pad_to_mask_clearance 0)
     (pcbplotparams
-      (layerselection 0x0001000_7fffffff)
+      (layerselection 0x0001000_fffffffe)
       (disableapertmacros false)
       (usegerberextensions false)
@@
   (gr_line (start 121 70) (end 121 108) (layer "Edge.Cuts") (width 0.1))
   (gr_line (start 28 70.006939) (end 28 108) (layer "Edge.Cuts") (width 0.1))
+  (gr_poly
+    (pts
+      (xy 121 118.75)
+      (xy 21.5 118.75)
+      (xy 21.5 59.5)
+      (xy 121 59.5)
+    ) (layer "Edge.Cuts") (width 0.1) (fill none))
   (gr_arc (start 28 108) (mid 31.181981 109.318019) (end 32.5 112.5) (layer "Edge.Cuts") (width 0.1))
-  (gr_arc (start 32.5 65.75) (mid 31.097238 68.774083) (end 28 70.006939) (layer "Edge.Cuts") (width 0.1))
+  (gr_arc (start 32.5 65.75) (mid 31.097021 68.773853) (end 28 70.006939) (layer "Edge.Cuts") (width 0.1))
   (gr_line (start 121 108) (end 108 108) (layer "Edge.Cuts") (width 0.1))
   (gr_line (start 103.5 112.5) (end 103.5 115) (layer "Edge.Cuts") (width 0.1))
@@
   )
   (via locked (at 39 109) (size 5) (drill 3) (layers "F.Cu" "B.Cu") (free) (net 0))
+  (via (at 108 112.5) (size 8.5) (drill 1) (layers "F.Cu" "B.Cu") (free) (net 0))
   (via locked (at 89 109) (size 5) (drill 3) (layers "F.Cu" "B.Cu") (free) (net 0))
+  (via (at 28 112.5) (size 8.5) (drill 1) (layers "F.Cu" "B.Cu") (free) (net 0))
   (via locked (at 89 69) (size 5) (drill 3) (layers "F.Cu" "B.Cu") (free) (net 0))
+  (via (at 28 65.5) (size 8.5) (drill 1) (layers "F.Cu" "B.Cu") (free) (net 0))
   (via locked (at 39 69) (size 5) (drill 3) (layers "F.Cu" "B.Cu") (free) (net 0))
+  (via (at 108 65.5) (size 8.5) (drill 1) (layers "F.Cu" "B.Cu") (free) (net 0))
   (segment (start 74.1375 99.425) (end 75.425 99.425) (width 0.4) (layer "F.Cu") (net 1))
   (segment (start 75.425 99.425) (end 75.75 99.75) (width 0.4) (layer "F.Cu") (net 1))
